File: NightLight_ESP32_tall.kicad_pcb (KiCad board)
At the start: 2 copper layers, 30 x 120 mm, 27 parts, among them J1 USB_C_Receptacle_USB2.0, J2 BUTTON, Q1 MMBT2222, Q2 MMBT2222, SW1 TL3342, SW2 TL3342, U1 ESP32-WROOM-32D, U2 AP2112K-3.3, U3 CH340C

Commit message: A few tweeks
Routing:
- net /D-: track 44.3 -> 52.9 mm, vias 2 -> 3
- net /D+: track 44.1 -> 51.4 mm, vias 2 -> 3
- net /NEOPIXEL: track 67.6 -> 66.2 mm
- net /DTR: track 12.4 -> 11.0 mm
- net /BUTTON: track 114.0 -> 112.9 mm
- net /RXD0: track 67.7 -> 68.5 mm
- net /TXD0: track 72.1 -> 72.9 mm
- net GND: track 42.5 -> 43.2 mm
- net /GPIO0: track 39.9 -> 40.4 mm

Commit message: Updated to v6
Other:
- net class Default removed
